Commit message: update

File: robotiq2f_description/urdf/robotiq85/robotiq_85_macro.urdf.xacro (robot description, xacro)
@@ -19,10 +19,10 @@
 			<visual> <!-- Gripper body -->
 				<geometry>
-					<mesh filename="package://robotiq2f_description/meshes/visual/robotiq_85_base_link.dae"/>
-				</geometry>
-			</visual>
-			<collision>
-				<geometry>
-					<mesh filename="package://robotiq2f_description/meshes/collision/robotiq_85_base_link.stl"/>
+					<mesh filename="package://robotiq2f_description/meshes/robotiq85/visual/robotiq_85_base_link.dae"/>
+				</geometry>
+			</visual>
+			<collision>
+				<geometry>
+					<mesh filename="package://robotiq2f_description/meshes/robotiq85/collision/robotiq_85_base_link.stl"/>
 				</geometry>
 			</collision>
@@ -55,10 +55,10 @@
 			<visual>
 				<geometry>
-					<mesh filename="package://robotiq2f_description/meshes/visual/robotiq_85_knuckle_link.dae"/>
-				</geometry>
-			</visual>
-			<collision>
-				<geometry>
-					<mesh filename="package://robotiq2f_description/meshes/collision/robotiq_85_knuckle_link.stl"/>
+					<mesh filename="package://robotiq2f_description/meshes/robotiq85/visual/robotiq_85_knuckle_link.dae"/>
+				</geometry>
+			</visual>
+			<collision>
+				<geometry>
+					<mesh filename="package://robotiq2f_description/meshes/robotiq85/collision/robotiq_85_knuckle_link.stl"/>
 				</geometry>
 			</collision>
@@ -74,10 +74,10 @@
 			<visual>
 				<geometry>
-					<mesh filename="package://robotiq2f_description/meshes/visual/robotiq_85_knuckle_link.dae"/>
-				</geometry>
-			</visual>
-			<collision>
-				<geometry>
-					<mesh filename="package://robotiq2f_description/meshes/collision/robotiq_85_knuckle_link.stl"/>
+					<mesh filename="package://robotiq2f_description/meshes/robotiq85/visual/robotiq_85_knuckle_link.dae"/>
+				</geometry>
+			</visual>
+			<collision>
+				<geometry>
+					<mesh filename="package://robotiq2f_description/meshes/robotiq85/collision/robotiq_85_knuckle_link.stl"/>
 				</geometry>
 			</collision>
@@ -103,10 +103,10 @@
 			<visual>
 				<geometry>
-					<mesh filename="package://robotiq2f_description/meshes/visual/robotiq_85_finger_link.dae"/>
-				</geometry>
-			</visual>
-			<collision>
-				<geometry>
-					<mesh filename="package://robotiq2f_description/meshes/collision/robotiq_85_finger_link.stl"/>
+					<mesh filename="package://robotiq2f_description/meshes/robotiq85/visual/robotiq_85_finger_link.dae"/>
+				</geometry>
+			</visual>
+			<collision>
+				<geometry>
+					<mesh filename="package://robotiq2f_description/meshes/robotiq85/collision/robotiq_85_finger_link.stl"/>
 				</geometry>
 			</collision>
@@ -122,10 +122,10 @@
 			<visual>
 				<geometry>
-					<mesh filename="package://robotiq2f_description/meshes/visual/robotiq_85_finger_link.dae"/>
-				</geometry>
-			</visual>
-			<collision>
-				<geometry>
-					<mesh filename="package://robotiq2f_description/meshes/collision/robotiq_85_finger_link.stl"/>
+					<mesh filename="package://robotiq2f_description/meshes/robotiq85/visual/robotiq_85_finger_link.dae"/>
+				</geometry>
+			</visual>
+			<collision>
+				<geometry>
+					<mesh filename="package://robotiq2f_description/meshes/robotiq85/collision/robotiq_85_finger_link.stl"/>
 				</geometry>
 			</collision>
@@ -157,10 +157,10 @@
 			<visual>
 				<geometry>
-					<mesh filename="package://robotiq2f_description/meshes/visual/robotiq_85_inner_knuckle_link.dae"/>
-				</geometry>
-			</visual>
-			<collision>
-				<geometry>
-					<mesh filename="package://robotiq2f_description/meshes/collision/robotiq_85_inner_knuckle_link.stl"/>
+					<mesh filename="package://robotiq2f_description/meshes/robotiq85/visual/robotiq_85_inner_knuckle_link.dae"/>
+				</geometry>
+			</visual>
+			<collision>
+				<geometry>
+					<mesh filename="package://robotiq2f_description/meshes/robotiq85/collision/robotiq_85_inner_knuckle_link.stl"/>
 				</geometry>
 			</collision>
@@ -176,10 +176,10 @@
 			<visual>
 				<geometry>
-					<mesh filename="package://robotiq2f_description/meshes/visual/robotiq_85_inner_knuckle_link.dae"/>
-				</geometry>
-			</visual>
-			<collision>
-				<geometry>
-					<mesh filename="package://robotiq2f_description/meshes/collision/robotiq_85_inner_knuckle_link.stl"/>
+					<mesh filename="package://robotiq2f_description/meshes/robotiq85/visual/robotiq_85_inner_knuckle_link.dae"/>
+				</geometry>
+			</visual>
+			<collision>
+				<geometry>
+					<mesh filename="package://robotiq2f_description/meshes/robotiq85/collision/robotiq_85_inner_knuckle_link.stl"/>
 				</geometry>
 			</collision>
@@ -211,10 +211,10 @@
 			<visual>
 				<geometry>
-					<mesh filename="package://robotiq2f_description/meshes/visual/robotiq_85_finger_tip_link.dae"/>
-				</geometry>
-			</visual>
-			<collision>
-				<geometry>
-					<mesh filename="package://robotiq2f_description/meshes/collision/robotiq_85_finger_tip_link.stl"/>
+					<mesh filename="package://robotiq2f_description/meshes/robotiq85/visual/robotiq_85_finger_tip_link.dae"/>
+				</geometry>
+			</visual>
+			<collision>
+				<geometry>
+					<mesh filename="package://robotiq2f_description/meshes/robotiq85/collision/robotiq_85_finger_tip_link.stl"/>
 				</geometry>
 			</collision>
@@ -230,10 +230,10 @@
 			<visual>
 				<geometry>
-					<mesh filename="package://robotiq2f_description/meshes/visual/robotiq_85_finger_tip_link.dae"/>
-				</geometry>
-			</visual>
-			<collision>
-				<geometry>
-					<mesh filename="package://robotiq2f_description/meshes/collision/robotiq_85_finger_tip_link.stl"/>
+					<mesh filename="package://robotiq2f_description/meshes/robotiq85/visual/robotiq_85_finger_tip_link.dae"/>
+				</geometry>
+			</visual>
+			<collision>
+				<geometry>
+					<mesh filename="package://robotiq2f_description/meshes/robotiq85/collision/robotiq_85_finger_tip_link.stl"/>
 				</geometry>
 			</collision>

File: robotiq2f_description/urdf/robotiq85/ur_to_robotiq_adapter.urdf.xacro (robot description, xacro)
@@ -12,5 +12,5 @@
 			<origin xyz="0 0 0" rpy="0 0 0" />
 			<geometry>
-				<mesh filename="package://robotiq2f_description/meshes/visual/ur_to_robotiq_adapter.dae"/>
+				<mesh filename="package://robotiq2f_description/meshes/robotiq85/visual/ur_to_robotiq_adapter.dae"/>
 			</geometry>
 		</visual>
@@ -18,5 +18,5 @@
 			<origin xyz="0 0 0" rpy="0 0 0"/>
 			<geometry>
-				<mesh filename="package://robotiq2f_description/meshes/collision/ur_to_robotiq_adapter.stl"/>
+				<mesh filename="package://robotiq2f_description/meshes/robotiq85/collision/ur_to_robotiq_adapter.stl"/>
 			</geometry>
 		</collision>
