Commit message: update

File: robotiq2f_description/urdf/robotiq85/robotiq_85_macro.xacro (robot description, xacro)
@@ -8,6 +8,25 @@
 		</joint>
 		<link name="${prefix}robotiq_85_base_link">
-			<visual>
-				<origin xyz="0.16 0 0" rpy="0 0 0" />
+			<visual> <!-- Gripper body -->
+				<geometry>
+					<mesh filename="package://robotiq2f_description/meshes/robotiq85/visual/robotiq_85_base_link.dae"/>
+				</geometry>
+			</visual>
+			<collision>
+				<geometry>
+					<mesh filename="package://robotiq2f_description/meshes/robotiq85/collision/robotiq_85_base_link.stl"/>
+				</geometry>
+			</collision>
+			<inertial>
+				<mass value="0.636951" />
+				<origin xyz="0.0 0.0 0.0" />
+				<inertia ixx = "0.000380" ixy = "0.000000" ixz = "0.000000"
+					iyx = "0.000000" iyy = "0.001110" iyz = "0.000000"
+					izx = "0.000000" izy = "0.000000" izz = "0.001171" />
+			</inertial>
+		</link>
+		<link name="${prefix}robotiq_85_tip">
+			<visual>
+				<origin xyz="0 0 0" rpy="0 0 0" />
 				<geometry>
 					<sphere radius="0.007"/> <!-- Visual aid for grasping sphere in front of gripper -->
@@ -17,22 +36,10 @@
 				</material>
 			</visual>
-			<visual> <!-- Gripper body -->
-				<geometry>
-					<mesh filename="package://robotiq2f_description/meshes/robotiq85/visual/robotiq_85_base_link.dae"/>
-				</geometry>
-			</visual>
-			<collision>
-				<geometry>
-					<mesh filename="package://robotiq2f_description/meshes/robotiq85/collision/robotiq_85_base_link.stl"/>
-				</geometry>
-			</collision>
-			<inertial>
-				<mass value="0.636951" />
-				<origin xyz="0.0 0.0 0.0" />
-				<inertia ixx = "0.000380" ixy = "0.000000" ixz = "0.000000"
-					iyx = "0.000000" iyy = "0.001110" iyz = "0.000000"
-					izx = "0.000000" izy = "0.000000" izz = "0.001171" />
-			</inertial>
-		</link>
+		</link>
+		<joint name="${prefix}robotiq_85_base_to_tip_joint" type="fixed">
+			<parent link="${prefix}robotiq_85_base_link"/>
+			<child link="${prefix}robotiq_85_tip"/>
+			<origin xyz="0.16 0 0" rpy="0 0 0" />
+		</joint>
 		<joint name="${prefix}robotiq_85_left_knuckle_joint" type="revolute">
 			<parent link="${prefix}robotiq_85_base_link"/>

File: robotiq2f_description/urdf/robotiqhande/robotiq_hande_macro.xacro (robot description, xacro)
@@ -1,5 +1,10 @@
 <?xml version="1.0"?>
 <robot xmlns:xacro="http://ros.org/wiki/xacro">
-	<xacro:macro name="robotiq_hande" params="prefix">
+	<xacro:macro name="robotiq_hande" params="prefix parent *origin">
+		<joint name="${prefix}robotiq_hande_base_joint" type="fixed">
+			<parent link="${parent}" />
+			<child link="${prefix}robotiq_hande_base_link" />
+			<xacro:insert_block name="origin" />
+		</joint>
 		<link name="${prefix}robotiq_hande_base_link">
 			<inertial>
@@ -12,5 +17,6 @@
 				<origin xyz="0 0 0" rpy="0 0 0" />
 				<geometry>
-					<mesh filename="package://robotiq2f_description/meshes/robotiqhande/visual/hand-e.dae"
+					<mesh
+						filename="package://robotiq2f_description/meshes/robotiqhande/visual/hand-e.dae"
 						scale="0.001 0.001 0.001" />
 				</geometry>
@@ -22,5 +28,6 @@
 				<origin xyz="0 0 0" rpy="0 0 0" />
 				<geometry>
-					<mesh filename="package://robotiq2f_description/meshes/robotiqhande/visual/hand-e.dae"
+					<mesh
+						filename="package://robotiq2f_description/meshes/robotiqhande/visual/hand-e.dae"
 						scale="0.001 0.001 0.001" />
 				</geometry>
@@ -37,5 +44,6 @@
 				<origin rpy="0 0 0" xyz="0 0 0" />
 				<geometry>
-					<mesh filename="package://robotiq2f_description/meshes/robotiqhande/visual/finger_1.dae"
+					<mesh
+						filename="package://robotiq2f_description/meshes/robotiqhande/visual/finger_1.dae"
 						scale="0.001 0.001 0.001" />
 				</geometry>
@@ -47,5 +55,6 @@
 				<origin rpy="0 0 0" xyz="0 0 0" />
 				<geometry>
-					<mesh filename="package://robotiq2f_description/meshes/robotiqhande/visual/finger_1.dae"
+					<mesh
+						filename="package://robotiq2f_description/meshes/robotiqhande/visual/finger_1.dae"
 						scale="0.001 0.001 0.001" />
 				</geometry>
@@ -62,5 +71,6 @@
 				<origin rpy="0 0 0" xyz="0 0 0" />
 				<geometry>
-					<mesh filename="package://robotiq2f_description/meshes/robotiqhande/visual/finger_2.dae"
+					<mesh
+						filename="package://robotiq2f_description/meshes/robotiqhande/visual/finger_2.dae"
 						scale="0.001 0.001 0.001" />
 				</geometry>
@@ -72,5 +82,6 @@
 				<origin rpy="0 0 0" xyz="0 0 0" />
 				<geometry>
-					<mesh filename="package://robotiq2f_description/meshes/robotiqhande/visual/finger_2.dae"
+					<mesh
+						filename="package://robotiq2f_description/meshes/robotiqhande/visual/finger_2.dae"
 						scale="0.001 0.001 0.001" />
 				</geometry>
